File: KiCad_FlashyHat.kicad_pcb (KiCad board)
At the start: 2 copper layers, 50 x 28.9 mm, 28 parts, among them J1 MK-12C02

Commit message: Fixed layout
Routing:
- net GND: track 79.4 -> 85.0 mm, vias 5 -> 7
- net Net-(D1-Pad2): track 97.5 -> 96.1 mm
- removed copper zone on B.Cu, net GND
- removed copper zone on F.Cu, net GND
Changed lines of the file:
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@@
   (segment (start 164.38548 98.85452) (end 164.38548 102.077973) (width 0.25) (layer "F.Cu") (net 2))
   (segment (start 168.35452 102.43452) (end 167.31 101.39) (width 0.25) (layer "F.Cu") (net 2))
+  (segment (start 143.04 98.01) (end 143.44 98.01) (width 0.25) (layer "F.Cu") (net 2))
   (segment (start 128.44 89.9) (end 128.44 91.489993) (width 0.25) (layer "F.Cu") (net 2))
   (segment (start 133.50548 92.92452) (end 134.42 92.01) (width 0.25) (layer "F.Cu") (net 2))
-  (segment (start 134.42 90.81) (end 136.9 88.33) (width 0.25) (layer "F.Cu") (net 2))
   (segment (start 134.42 92.01) (end 134.42 90.81) (width 0.25) (layer "F.Cu") (net 2))
   (segment (start 128.44 91.489993) (end 129.874527 92.92452) (width 0.25) (layer "F.Cu") (net 2))
@@
   (segment (start 128.8 84.64) (end 127.43798 86.00202) (width 0.25) (layer "F.Cu") (net 2))
   (segment (start 145.02452 95.21548) (end 152.29548 95.21548) (width 0.25) (layer "F.Cu") (net 2))
+  (segment (start 142.350489 89.456193) (end 142.350489 91.999511) (width 0.25) (layer "F.Cu") (net 2))
   (segment (start 171.840473 102.43452) (end 168.35452 102.43452) (width 0.25) (layer "F.Cu") (net 2))
   (segment (start 136.99 98.95) (end 138.32 100.28) (width 0.25) (layer "F.Cu") (net 2))
   (segment (start 127.43798 86.00202) (end 127.43798 88.89798) (width 0.25) (layer "F.Cu") (net 2))
-  (segment (start 136.9 88.33) (end 142.5 88.33) (width 0.25) (layer "F.Cu") (net 2))
-  (segment (start 143.31 89.14) (end 143.31 91.04) (width 0.25) (layer "F.Cu") (net 2))
-  (segment (start 143.31 91.04) (end 140.61 93.74) (width 0.25) (layer "F.Cu") (net 2))
+  (segment (start 142.350489 91.999511) (end 140.61 93.74) (width 0.25) (layer "F.Cu") (net 2))
+  (segment (start 143.44 98.01) (end 144.71 99.28) (width 0.25) (layer "F.Cu") (net 2))
   (segment (start 164.58 97.74) (end 164.58 98.66) (width 0.25) (layer "F.Cu") (net 2))
-  (segment (start 142.5 88.33) (end 143.31 89.14) (width 0.25) (layer "F.Cu") (net 2))
   (segment (start 143.04 97.2) (end 143.99 96.25) (width 0.25) (layer "F.Cu") (net 2))
+  (segment (start 136.09 89.14) (end 142.034296 89.14) (width 0.25) (layer "F.Cu") (net 2))
   (segment (start 163.648933 102.81452) (end 160.76452 102.81452) (width 0.25) (layer "F.Cu") (net 2))
   (segment (start 152.29548 95.21548) (end 152.55 95.47) (width 0.25) (layer "F.Cu") (net 2))
   (segment (start 129.874527 92.92452) (end 133.50548 92.92452) (width 0.25) (layer "F.Cu") (net 2))
+  (segment (start 142.034296 89.14) (end 142.350489 89.456193) (width 0.25) (layer "F.Cu") (net 2))
   (segment (start 127.43798 88.89798) (end 128.44 89.9) (width 0.25) (layer "F.Cu") (net 2))
+  (segment (start 134.42 90.81) (end 136.09 89.14) (width 0.25) (layer "F.Cu") (net 2))
   (segment (start 136.49 98.95) (end 136.99 98.95) (width 0.25) (layer "F.Cu") (net 2))
   (segment (start 173.23 98.47) (end 173.23 101.044993) (width 0.25) (layer "F.Cu") (net 2))
@@
   (via (at 136.49 98.95) (size 0.8) (drill 0.4) (layers "F.Cu" "B.Cu") (net 2))
   (via (at 154.9 87.04) (size 0.8) (drill 0.4) (layers "F.Cu" "B.Cu") (net 2))
+  (via (at 159.74 101.79) (size 0.8) (drill 0.4) (layers "F.Cu" "B.Cu") (net 2))
+  (via (at 152.55 95.47) (size 0.8) (drill 0.4) (layers "F.Cu" "B.Cu") (net 2))
   (via (at 140.61 93.74) (size 0.8) (drill 0.4) (layers "F.Cu" "B.Cu") (net 2))
   (via (at 143.04 98.01) (size 0.8) (drill 0.4) (layers "F.Cu" "B.Cu") (net 2))
@@
   (segment (start 138.259022 98.95) (end 136.49 98.95) (width 0.25) (layer "B.Cu") (net 2))
   (segment (start 140.61 93.74) (end 140.61 96.599022) (width 0.25) (layer "B.Cu") (net 2))
+  (segment (start 154.51 100.79) (end 158.74 100.79) (width 0.25) (layer "B.Cu") (net 2))
+  (segment (start 158.74 100.79) (end 159.74 101.79) (width 0.25) (layer "B.Cu") (net 2))
   (segment (start 130.8 84.64) (end 132.3875 84.64) (width 0.25) (layer "F.Cu") (net 3))
   (segment (start 132.3875 84.64) (end 132.7375 84.29) (width 0.25) (layer "F.Cu") (net 3))
-  (segment (start 142.796194 87.88049) (end 143.739511 88.823807) (width 0.25) (layer "F.Cu") (net 4))
   (segment (start 146.725 101.31) (end 149.43 101.31) (width 0.25) (layer "F.Cu") (net 4))
-  (segment (start 143.759511 88.953807) (end 143.759511 94.717989) (width 0.25) (layer "F.Cu") (net 4))
-  (segment (start 143.739511 88.823807) (end 143.739511 88.933807) (width 0.25) (layer "F.Cu") (net 4))
   (segment (start 157.107973 101.81452) (end 153.60952 101.81452) (width 0.25) (layer "F.Cu") (net 4))
   (segment (start 172.15452 100.53298) (end 171.2775 101.41) (width 0.25) (layer "F.Cu") (net 4))
   (segment (start 160.434993 95.49) (end 161.7675 96.822507) (width 0.25) (layer "F.Cu") (net 4))
+  (segment (start 142.81 89.28) (end 142.81 93.768478) (width 0.25) (layer "F.Cu") (net 4))
+  (segment (start 143.759511 94.717989) (end 140.3375 98.14) (width 0.25) (layer "F.Cu") (net 4))
   (segment (start 166.87202 95.35548) (end 172.27298 95.35548) (width 0.25) (layer "F.Cu") (net 4))
   (segment (start 151.58048 101.83452) (end 152.605 100.81) (width 0.25) (layer "F.Cu") (net 4))
@@
   (segment (start 146.725 101.31) (end 145.70048 102.33452) (width 0.25) (layer "F.Cu") (net 4))
   (segment (start 163.994527 94.59548) (end 165.58298 94.59548) (width 0.25) (layer "F.Cu") (net 4))
-  (segment (start 143.759511 94.717989) (end 140.3375 98.14) (width 0.25) (layer "F.Cu") (net 4))
   (segment (start 158.4275 95.49) (end 160.434993 95.49) (width 0.25) (layer "F.Cu") (net 4))
   (segment (start 131.3675 87.71) (end 130.3875 87.71) (width 0.25) (layer "F.Cu") (net 4))
+  (segment (start 132.375 91.242507) (end 134.988753 88.628753) (width 0.25) (layer "F.Cu") (net 4))
   (segment (start 158.4275 100.494993) (end 157.107973 101.81452) (width 0.25) (layer "F.Cu") (net 4))
+  (segment (start 134.988753 88.628753) (end 142.158753 88.628753) (width 0.25) (layer "F.Cu") (net 4))
   (segment (start 166.6075 95.62) (end 166.87202 95.35548) (width 0.25) (layer "F.Cu") (net 4))
   (segment (start 149.65548 96.53452) (end 149.65548 101.53548) (width 0.25) (layer "F.Cu") (net 4))
-  (segment (start 135.737017 87.88049) (end 142.796194 87.88049) (width 0.25) (layer "F.Cu") (net 4))
   (segment (start 149.95 96.24) (end 149.65548 96.53452) (width 0.25) (layer "F.Cu") (net 4))
+  (segment (start 142.81 93.768478) (end 143.759511 94.717989) (width 0.25) (layer "F.Cu") (net 4))
   (segment (start 149.43 101.31) (end 149.65548 101.53548) (width 0.25) (layer "F.Cu") (net 4))
   (segment (start 131.3675 87.71) (end 134.7875 84.29) (width 0.25) (layer "F.Cu") (net 4))
   (segment (start 165.58298 94.59548) (end 166.6075 95.62) (width 0.25) (layer "F.Cu") (net 4))
   (segment (start 161.7675 99.68) (end 161.7675 96.822507) (width 0.25) (layer "F.Cu") (net 4))
+  (segment (start 142.158753 88.628753) (end 142.81 89.28) (width 0.25) (layer "F.Cu") (net 4))
   (segment (start 144.06452 102.33452) (end 140.3375 98.6075) (width 0.25) (layer "F.Cu") (net 4))
   (segment (start 132.375 90.535) (end 131.58 89.74) (width 0.25) (layer "F.Cu") (net 4))
-  (segment (start 143.739511 88.933807) (end 143.759511 88.953807) (width 0.25) (layer "F.Cu") (net 4))
   (segment (start 173.2975 96.38) (end 172.15452 97.52298) (width 0.25) (layer "F.Cu") (net 4))
-  (segment (start 132.375 91.242507) (end 135.737017 87.88049) (width 0.25) (layer "F.Cu") (net 4))
   (via (at 140.3375 98.14) (size 0.8) (drill 0.4) (layers "F.Cu" "B.Cu") (net 4))
   (segment (start 137.249617 100.826102) (end 139.935719 98.14) (width 0.25) (layer "B.Cu") (net 4))
@@
   (segment (start 171.2475 98.4525) (end 171.23 98.47) (width 0.25) (layer "F.Cu") (net 15))
   (segment (start 171.2475 96.38) (end 171.2475 98.4525) (width 0.25) (layer "F.Cu") (net 15))
-  (zone (net 2) (net_name "GND") (layer "F.Cu") (hatch edge 0.508)
-    (connect_pads (clearance 0.508))
-    (min_thickness 0.254) (filled_areas_thickness no)
-    (fill yes (thermal_gap 0.508) (thermal_bridge_width 0.508))
-    (polygon
-      (pts
-        (xy 158.82 74.21)
-        (xy 178.76 91.97)
-        (xy 177.73 105.84)
-        (xy 171.65 111.19)
-        (xy 132.54 109.79)
-        (xy 122.08 94.77)
-        (xy 120.62 73.24)
-      )
-    )
-  )
-  (zone (net 2) (net_name "GND") (layer "B.Cu") (hatch edge 0.508)
-    (connect_pads (clearance 0.508))
-    (min_thickness 0.254) (filled_areas_thickness no)
-    (fill yes (thermal_gap 0.508) (thermal_bridge_width 0.508))
-    (polygon
-      (pts
-        (xy 170.76 78.25)
-        (xy 171.67 81.63)
-        (xy 181.25 93.67)
-        (xy 180.15 108.72)
-        (xy 156.07 113.56)
-        (xy 131.53 108.63)
-        (xy 125.14 95.95)
-        (xy 122.13 84.82)
-        (xy 130.43 75.33)
-        (xy 151.32 72.96)
-      )
-    )
-  )
   (group "" (id 0839ce8d-bc94-4a18-9387-0ce4b277e1aa)
     (members

Commit message: Fixed position ordernr
Other:
- board text added: "JLCJLCJLCJLC"
Changed lines of the file:
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@@
   (gr_curve (pts (xy 132.050433 94.136155) (xy 131.77647 94.096758) (xy 131.544606 94.072242) (xy 131.535179 94.081666)) (layer "Edge.Cuts") (width 0.2))
   (gr_curve (pts (xy 125.920488 87.9397) (xy 126.113692 87.182998) (xy 126.504982 86.248043) (xy 126.871372 85.667643)) (layer "Edge.Cuts") (width 0.2))
+  (gr_text "JLCJLCJLCJLC" (at 145.46 81.7 26) (layer "B.SilkS")
+    (effects (font (size 0.9 0.9) (thickness 0.225)) (justify mirror))
+  )
   (segment (start 165.33 91.43) (end 165.33 94) (width 0.25) (layer "B.Cu") (net 1))
   (segment (start 143.340099 98.734501) (end 143.764501 98.310099) (width 0.25) (layer "B.Cu") (net 1))
